File: Flight Computer/wiring/WYVERN_E4_flight_wiring_connected.kicad_sch (KiCad schematic)
At the start: 0 parts

Commit message: Commit!
Other:
- note added: "ADC_NODE"
- note added: "GP26 VBAT"
- note added: "R_top 100k / R_bot 62k -> 0.3827"
- note added: "VBAT DIVIDER"
- note added: "VBAT_TAP"
- note added: "WYVERN-E — Flight Wiring (fully routed, all components connected)"
- note removed: "WYVERN-E 4.0 — Flight Wiring (fully routed, all components connected)"
- title: WYVERN-E 4.0 Flight Wiring — fully routed -> WYVERN-E Flight Wiring — fully routed

Commit message: Update - but the PCB no work :(
Other:
- note added: "+V"
- note added: "3V3IN"
- note added: "7.4V -> VBUCK"
- note added: "A1"
- note added: "AP2112K-3.3 LDO (U7)"
- note added: "BME680 0x76"
- note added: "BNO055 BODY 0x28"
- note added: "BNO085 EXTERNAL 0x4A"
- note added: "GP0 SDA0"
- note added: "GP1 SCL0"
- note added: "GP10 SCK"
- note added: "GP11 MOSI"
- note added: "GP12 RBF"
- note added: "GP2 S1"
- note added: "GP3 S2"
- note added: "GP34 BUZ"
- note added: "GP35 LED"
- note added: "GP36 CAM"
- note added: "GP37 IRQ"
- note added: "GP4 spare"
- note added: "GP5 spare"
- note added: "GP8 MISO"
- note added: "GP9 CS"
- note added: "INA226 (U4) -- WIRING PROBLEM"
- note added: "LIS3MDL (U5) 0x1C"
- note added: "One shared I2C bus (no mux), every address netlist-CONFIRMED: body BNO055 0x28, external BNO085 0x4A (STEMMA-QT, bulkhead-boundary mount), BME680 0x76, LIS3MDL 0x1C. No BMP388 populated, no WiFi/BLE radio chip on this board. INA226 (U4) has a real wiring problem, not just an unverified address -- reads the ~5V buck rail instead of pack voltage, no true current shunt, address strap ties to an inva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"
- note added: "QFN-80 · dual-M33 · no radio chip"
- note added: "R10 (10mOhm, 2512) -- parallel w/ SW U13, not a shunt"
- note added: "RP2350B (U1)"
- note added: "SERVO 1 (pitch, JST U8)"
- note added: "SERVO 2 (yaw, JST U9)"
- note added: "STEMMA-QT · bulkhead-boundary mount, not gimbal"
- note added: "TPS564201 BUCK (U15)"
- note added: "VBUCK"
- note added: "VBUCK -> 3.3V"
- note added: "VBUS"
- note added: "VIN+"
- note added: "VIN-"
- note added: "V_EN"
- note added: "WYVERN-E, Flight Wiring (fully routed, all components connected) -- PCB1 custom RP2350B"
- note added: "addr CONFIRMED (SD0/SA1->GND) · unused by firmware"
- note added: "flight log · pin4/VDD traces to GND, possible defect"
- note added: "microSD (CARD1)"
- note added: "onboard baro · addr CONFIRMED (SDO->GND)"
- note added: "onboard · addr CONFIRMED (COM3->GND)"
- note added: "reads VBUCK not pack V; addr strap invalid, see CONFLICTS.md"
- note added: "to VBUCK"
- note removed: "+5V"
- note removed: "3V3OUT"
- note removed: "5V -> Pico+cam+servos"
- note removed: "ADC_NODE"
- note removed: "All sensors GRV (mag off). 3 BNO085 @0x4A: gimbal on dedicated I2C1; body/recovery isolated on PCA9548A ch0/ch1. RP2350 is 3.3V logic; all STEMMA-QT sensors (incl. BMP388) run at 3.3V."
- note removed: "BME688 0x76"
- note removed: "BMP388 0x77 (3966)"
- note removed: "BNO085 BODY 0x4A"
- note removed: "BNO085 GIMBAL 0x4A"
- note removed: "BNO085 RECOVERY 0x4A"
- note removed: "GP1 spare"
- note removed: "GP10 BUZ"
- note removed: "GP14 S1"
- note removed: "GP15 S2"
- note removed: "GP16 SDA0"
- note removed: "GP17 SCL0"
- note removed: "GP18 SDA1"
- note removed: "GP19 SCL1"
- note removed: "GP2 SCK"
- note removed: "GP22 RBF"
- note removed: "GP26 VBAT"
- note removed: "GP3 MOSI"
- note removed: "GP4 MISO"
- note removed: "GP5 CS"
- note removed: "GP6 spare"
- note removed: "GP7 IRQ"
- note removed: "GP8 CAM"
- note removed: "GP9 LED"
- note removed: "I2C0 trunk -> 5 ch"
- note removed: "I2C1 · GRV"
- note removed: "INT"
- note removed: "PCA9548A MUX 0x70"
- note removed: "RP2350 dual-M33 150MHz · WiFi/BLE"
- note removed: "RPi PICO 2 W"
- note removed: "R_top 100k / R_bot 62k -> 0.3827"
- note removed: "SERVO 1 (pitch)"
- note removed: "SERVO 2 (yaw)"
- note removed: "SW+fuse / 5V UBEC"
- note removed: "V5_EN"
- note removed: "VBAT DIVIDER"
- note removed: "VBAT_TAP"
- note removed: "VSYS"
- note removed: "WYVERN-E — Flight Wiring (fully routed, all components connected)"
- note removed: "c0 SC"
- note removed: "c0 SD"
- note removed: "c1 SC"
- note removed: "c1 SD"
- note removed: "c2 SC"
- note removed: "c2 SD"
- note removed: "c3 SC"
- note removed: "c3 SD"
- note removed: "flight log"
- note removed: "microSD (SPI0)"
- note removed: "mux c0 · GRV"
- note removed: "mux c1 · vote"
- note removed: "mux c2"
- note removed: "mux c3 · 3V3"
- title: WYVERN-E Flight Wiring — fully routed -> WYVERN-E Flight Wiring, fully routed

Commit message: Update!
Other:
- note added: "GTR70E WYVERN, Flight Wiring (fully routed, all components connected) -- PCB1 custom RP2350B"
- note removed: "WYVERN-E, Flight Wiring (fully routed, all components connected) -- PCB1 custom RP2350B"
- company: Skylight Rocketry -> Skylight Industries
- title: WYVERN-E Flight Wiring, fully routed -> GTR70E WYVERN Flight Wiring, fully routed
Changed lines of the file:
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@@
-(kicad_sch (version 20230121) (generator "wyvern4_connected") (paper "A1")
-  (title_block (title "WYVERN-E Flight Wiring, fully routed") (company "Skylight Rocketry") (rev "5.0"))
+(kicad_sch (version 20230121) (generator "gtr70e_wyvern_connected") (paper "A1")
+  (title_block (title "GTR70E WYVERN Flight Wiring, fully routed") (company "Skylight Industries") (rev "5.0"))
   (wire (pts (xy 40 18) (xy 395 18)) (stroke (width 0.3)(type solid)))
  (label "+VBUCK" (at 32 17.4 0)(effects (font (size 1.3 1.3))(justify left)))
@@
  (wire (pts (xy 157.0 60.0) (xy 157.0 286)) (stroke (width 0.15)(type solid)))
  (junction (at 157.0 286) (diameter 0.9) (color 0 0 0 0))
- (text "WYVERN-E, Flight Wiring (fully routed, all components connected) -- PCB1 custom RP2350B" (at 40 8 0)(effects (font (size 2.4 2.4))(justify left)))
+ (text "GTR70E WYVERN, Flight Wiring (fully routed, all components connected) -- PCB1 custom RP2350B" (at 40 8 0)(effects (font (size 2.4 2.4))(justify left)))
  (text "One shared I2C bus (no mux), every address netlist-CONFIRMED: body BNO055 0x28, external BNO085 0x4A (STEMMA-QT, bulkhead-boundary mount), BME680 0x76, LIS3MDL 0x1C. No BMP388 populated, no WiFi/BLE radio chip on this board. INA226 (U4) has a real wiring problem, not just an unverified address -- reads the ~5V buck rail instead of pack voltage, no true current shunt, address strap ties to an invalid ~5V node -- see CONFLICTS.md section 3 and battery.h. RBF (GP12/H1 pin13) is not wired to any switch on this board rev; the other four H1 GPIOs (37/36/35/34) are confirmed-usable, their function assignment is a firmware choice. CARD1 pin4 traces to GND where VDD would be expected -- possible SD-power defect, bench-check before trusting flight logging." (at 40 300 0)(effects (font (size 1.1 1.1))(justify left)))
   (sheet_instances (path "/" (page "1"))))
