File: Flight Computer/wiring/WYVERN_E4_tvc_balance_harness.kicad_sch (KiCad schematic)
At the start: 0 parts

Commit message: Update!
Other:
- company: Skylight Rocketry -> Skylight Industries
- title: WYVERN-E 4.0 — 3-axis TVC balance harness -> GTR70E WYVERN 4.0 — 3-axis TVC balance harness
Changed lines of the file:
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@@
-(kicad_sch (version 20230121) (generator "wyvern4_wiring") (paper "A2")
-  (title_block (title "WYVERN-E 4.0 — 3-axis TVC balance harness") (company "Skylight Rocketry") (rev "4.0"))
+(kicad_sch (version 20230121) (generator "gtr70e_wyvern_wiring") (paper "A2")
+  (title_block (title "GTR70E WYVERN 4.0 — 3-axis TVC balance harness") (company "Skylight Industries") (rev "4.0"))
   (rectangle (start 20 20) (end 78 50) (stroke (width 0.25)(type solid)) (fill (type none)))
   (text "3-AXIS TVC BALANCE — DAQ (Arduino Nano)" (at 22 23 0)(effects (font (size 1.6 1.6))(justify left)))
