File: Flight Computer/wiring/WYVERN_E4_tvc_balance_servo_harness.kicad_sch (KiCad schematic)
At the start: 0 parts

Commit message: Commit!
Other:
- title: WYVERN-E 4.0 — TVC balance harness (servo rig, Pico) -> WYVERN-E — TVC balance harness (servo rig, Pico)
Changed lines of the file:
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@@
 (kicad_sch (version 20230121) (generator "wyvern4_wiring") (paper "A2")
-  (title_block (title "WYVERN-E 4.0 — TVC balance harness (servo rig, Pico)") (company "Skylight Rocketry") (rev "4.0"))
+  (title_block (title "WYVERN-E — TVC balance harness (servo rig, Pico)") (company "Skylight Rocketry") (rev "4.0"))
   (rectangle (start 20 20) (end 84 54) (stroke (width 0.25)(type solid)) (fill (type none)))
   (text "RPi PICO / PICO 2 W — servo-rig DAQ" (at 22 23 0)(effects (font (size 1.6 1.6))(justify left)))

Commit message: Update - but the PCB no work :(
Other:
- note added: "RPi PICO / PICO 2 W, servo-rig DAQ"
- note removed: "RPi PICO / PICO 2 W — servo-rig DAQ"
- title: WYVERN-E — TVC balance harness (servo rig, Pico) -> WYVERN-E, TVC balance harness (servo rig, Pico)
Changed lines of the file:
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@@
 (kicad_sch (version 20230121) (generator "wyvern4_wiring") (paper "A2")
-  (title_block (title "WYVERN-E — TVC balance harness (servo rig, Pico)") (company "Skylight Rocketry") (rev "4.0"))
+  (title_block (title "WYVERN-E, TVC balance harness (servo rig, Pico)") (company "Skylight Rocketry") (rev "4.0"))
   (rectangle (start 20 20) (end 84 54) (stroke (width 0.25)(type solid)) (fill (type none)))
-  (text "RPi PICO / PICO 2 W — servo-rig DAQ" (at 22 23 0)(effects (font (size 1.6 1.6))(justify left)))
-  (text "3V3: HX711 + BNO085 power" (at 22 28 0)(effects (font (size 1.2 1.2))(justify left)))
-  (global_label "3V3" (shape input)(at 84 28 0)(effects (font (size 1.0 1.0))(justify left)))
-  (wire (pts (xy 83 28) (xy 84 28)) (stroke (width 0.15)(type solid)))
-  (text "GND" (at 22 32 0)(effects (font (size 1.2 1.2))(justify left)))
-  (global_label "GND" (shape input)(at 84 32 0)(effects (font (size 1.0 1.0))(justify left)))
-  (wire (pts (xy 83 32) (xy 84 32)) (stroke (width 0.15)(type solid)))
-  (text "USB: CSV log to host" (at 22 36 0)(effects (font (size 1.2 1.2))(justify left)))
-  (global_label "USB" (shape input)(at 84 36 0)(effects (font (size 1.0 1.0))(justify left)))
-  (wire (pts (xy 83 36) (xy 84 36)) (stroke (width 0.15)(type solid)))
-  (text "GP4/GP5: I2C0 -> gimbal BNO085 (0x4A)" (at 22 40 0)(effects (font (size 1.2 1.2))(justify left)))
-  (global_label "GP4/GP5" (shape input)(at 84 40 0)(effects (font (size 1.0 1.0))(justify left)))
-  (wire (pts (xy 83 40) (xy 84 40)) (stroke (width 0.15)(type solid)))
-  (text "GP14: PWM servo1 (pitch)" (at 22 44 0)(effects (font (size 1.2 1.2))(justify left)))
-  (global_label "GP14" (shape input)(at 84 44 0)(effects (font (size 1.0 1.0))(justify left)))
-  (wire (pts (xy 83 44) (xy 84 44)) (stroke (width 0.15)(type solid)))
-  (text "GP15: PWM servo2 (yaw)" (at 22 48 0)(effects (font (size 1.2 1.2))(justify left)))
-  (global_label "GP15" (shape input)(at 84 48 0)(effects (font (size 1.0 1.0))(justify left)))
-  (wire (pts (xy 83 48) (xy 84 48)) (stroke (width 0.15)(type solid)))
-  (text "LED_BUILTIN: tare-complete blink" (at 22 52 0)(effects (font (size 1.2 1.2))(justify left)))
-  (global_label "LED_BUILTIN" (shape input)(at 84 52 0)(effects (font (size 1.0 1.0))(justify left)))
-  (wire (pts (xy 83 52) (xy 84 52)) (stroke (width 0.15)(type solid)))
-  (rectangle (start 20 62) (end 76 80) (stroke (width 0.25)(type solid)) (fill (type none)))
-  (text "LOAD CELLS + HX711 x3 (bit-banged)" (at 22 65 0)(effects (font (size 1.6 1.6))(justify left)))
-  (text "Z (axial, 5kg): DT GP10 / SCK GP11" (at 22 70 0)(effects (font (size 1.2 1.2))(justify left)))
-  (global_label "Z (axial, 5kg)" (shape input)(at 76 70 0)(effects (font (size 1.0 1.0))(justify left)))
-  (wire (pts (xy 75 70) (xy 76 70)) (stroke (width 0.15)(type solid)))
-  (text "X (lateral, 1kg): DT GP6 / SCK GP7" (at 22 74 0)(effects (font (size 1.2 1.2))(justify left)))
-  (global_label "X (lateral, 1kg)" (shape input)(at 76 74 0)(effects (font (size 1.0 1.0))(justify left)))
-  (wire (pts (xy 75 74) (xy 76 74)) (stroke (width 0.15)(type solid)))
-  (text "Y (lateral, 1kg): DT GP8 / SCK GP9" (at 22 78 0)(effects (font (size 1.2 1.2))(justify left)))
-  (global_label "Y (lateral, 1kg)" (shape input)(at 76 78 0)(effects (font (size 1.0 1.0))(justify left)))
-  (wire (pts (xy 75 78) (xy 76 78)) (stroke (width 0.15)(type solid)))
-  (rectangle (start 20 88) (end 72 98) (stroke (width 0.25)(type solid)) (fill (type none)))
-  (text "GIMBAL BNO085 (Game Rotation Vector)" (at 22 91 0)(effects (font (size 1.6 1.6))(justify left)))
-  (text "I2C0 0x4A: nozzle-angle cross-check vs. commanded servo pos" (at 22 96 0)(effects (font (size 1.2 1.2))(justify left)))
-  (global_label "I2C0 0x4A" (shape input)(at 72 96 0)(effects (font (size 1.0 1.0))(justify left)))
-  (wire (pts (xy 71 96) (xy 72 96)) (stroke (width 0.15)(type solid)))
-  (rectangle (start 20 106) (end 70 128) (stroke (width 0.25)(type solid)) (fill (type none)))
-  (text "SERVO GIMBAL UNDER TEST" (at 22 109 0)(effects (font (size 1.6 1.6))(justify left)))
-  (text "S1_SIG: GP14 (pitch)" (at 22 114 0)(effects (font (size 1.2 1.2))(justify left)))
-  (global_label "S1_SIG" (shape input)(at 70 114 0)(effects (font (size 1.0 1.0))(justify left)))
-  (wire (pts (xy 69 114) (xy 70 114)) (stroke (width 0.15)(type solid)))
-  (text "S2_SIG: GP15 (yaw)" (at 22 118 0)(effects (font (size 1.2 1.2))(justify left)))
-  (global_label "S2_SIG" (shape input)(at 70 118 0)(effects (font (size 1.0 1.0))(justify left)))
-  (wire (pts (xy 69 118) (xy 70 118)) (stroke (width 0.15)(type solid)))
-  (text "VSERVO" (at 22 122 0)(effects (font (size 1.2 1.2))(justify left)))
-  (global_label "VSERVO" (shape input)(at 70 122 0)(effects (font (size 1.0 1.0))(justify left)))
-  (wire (pts (xy 69 122) (xy 70 122)) (stroke (width 0.15)(type solid)))
-  (text "GND" (at 22 126 0)(effects (font (size 1.2 1.2))(justify left)))
-  (global_label "GND" (shape input)(at 70 126 0)(effects (font (size 1.0 1.0))(justify left)))
-  (wire (pts (xy 69 126) (xy 70 126)) (stroke (width 0.15)(type solid)))
+ (text "RPi PICO / PICO 2 W, servo-rig DAQ" (at 22 23 0)(effects (font (size 1.6 1.6))(justify left)))
+ (text "3V3: HX711 + BNO085 power" (at 22 28 0)(effects (font (size 1.2 1.2))(justify left)))
+ (global_label "3V3" (shape input)(at 84 28 0)(effects (font (size 1.0 1.0))(justify left)))
+ (wire (pts (xy 83 28) (xy 84 28)) (stroke (width 0.15)(type solid)))
+ (text "GND" (at 22 32 0)(effects (font (size 1.2 1.2))(justify left)))
+ (global_label "GND" (shape input)(at 84 32 0)(effects (font (size 1.0 1.0))(justify left)))
+ (wire (pts (xy 83 32) (xy 84 32)) (stroke (width 0.15)(type solid)))
+ (text "USB: CSV log to host" (at 22 36 0)(effects (font (size 1.2 1.2))(justify left)))
+ (global_label "USB" (shape input)(at 84 36 0)(effects (font (size 1.0 1.0))(justify left)))
+ (wire (pts (xy 83 36) (xy 84 36)) (stroke (width 0.15)(type solid)))
+ (text "GP4/GP5: I2C0 -> gimbal BNO085 (0x4A)" (at 22 40 0)(effects (font (size 1.2 1.2))(justify left)))
+ (global_label "GP4/GP5" (shape input)(at 84 40 0)(effects (font (size 1.0 1.0))(justify left)))
+ (wire (pts (xy 83 40) (xy 84 40)) (stroke (width 0.15)(type solid)))
+ (text "GP14: PWM servo1 (pitch)" (at 22 44 0)(effects (font (size 1.2 1.2))(justify left)))
+ (global_label "GP14" (shape input)(at 84 44 0)(effects (font (size 1.0 1.0))(justify left)))
+ (wire (pts (xy 83 44) (xy 84 44)) (stroke (width 0.15)(type solid)))
+ (text "GP15: PWM servo2 (yaw)" (at 22 48 0)(effects (font (size 1.2 1.2))(justify left)))
+ (global_label "GP15" (shape input)(at 84 48 0)(effects (font (size 1.0 1.0))(justify left)))
+ (wire (pts (xy 83 48) (xy 84 48)) (stroke (width 0.15)(type solid)))
+ (text "LED_BUILTIN: tare-complete blink" (at 22 52 0)(effects (font (size 1.2 1.2))(justify left)))
+ (global_label "LED_BUILTIN" (shape input)(at 84 52 0)(effects (font (size 1.0 1.0))(justify left)))
+ (wire (pts (xy 83 52) (xy 84 52)) (stroke (width 0.15)(type solid)))
+ (rectangle (start 20 62) (end 76 80) (stroke (width 0.25)(type solid)) (fill (type none)))
+ (text "LOAD CELLS + HX711 x3 (bit-banged)" (at 22 65 0)(effects (font (size 1.6 1.6))(justify left)))
+ (text "Z (axial, 5kg): DT GP10 / SCK GP11" (at 22 70 0)(effects (font (size 1.2 1.2))(justify left)))
+ (global_label "Z (axial, 5kg)" (shape input)(at 76 70 0)(effects (font (size 1.0 1.0))(justify left)))
+ (wire (pts (xy 75 70) (xy 76 70)) (stroke (width 0.15)(type solid)))
+ (text "X (lateral, 1kg): DT GP6 / SCK GP7" (at 22 74 0)(effects (font (size 1.2 1.2))(justify left)))
+ (global_label "X (lateral, 1kg)" (shape input)(at 76 74 0)(effects (font (size 1.0 1.0))(justify left)))
+ (wire (pts (xy 75 74) (xy 76 74)) (stroke (width 0.15)(type solid)))
+ (text "Y (lateral, 1kg): DT GP8 / SCK GP9" (at 22 78 0)(effects (font (size 1.2 1.2))(justify left)))
+ (global_label "Y (lateral, 1kg)" (shape input)(at 76 78 0)(effects (font (size 1.0 1.0))(justify left)))
+ (wire (pts (xy 75 78) (xy 76 78)) (stroke (width 0.15)(type solid)))
+ (rectangle (start 20 88) (end 72 98) (stroke (width 0.25)(type solid)) (fill (type none)))
+ (text "GIMBAL BNO085 (Game Rotation Vector)" (at 22 91 0)(effects (font (size 1.6 1.6))(justify left)))
+ (text "I2C0 0x4A: nozzle-angle cross-check vs. commanded servo pos" (at 22 96 0)(effects (font (size 1.2 1.2))(justify left)))
+ (global_label "I2C0 0x4A" (shape input)(at 72 96 0)(effects (font (size 1.0 1.0))(justify left)))
+ (wire (pts (xy 71 96) (xy 72 96)) (stroke (width 0.15)(type solid)))
+ (rectangle (start 20 106) (end 70 128) (stroke (width 0.25)(type solid)) (fill (type none)))
+ (text "SERVO GIMBAL UNDER TEST" (at 22 109 0)(effects (font (size 1.6 1.6))(justify left)))
+ (text "S1_SIG: GP14 (pitch)" (at 22 114 0)(effects (font (size 1.2 1.2))(justify left)))
+ (global_label "S1_SIG" (shape input)(at 70 114 0)(effects (font (size 1.0 1.0))(justify left)))
+ (wire (pts (xy 69 114) (xy 70 114)) (stroke (width 0.15)(type solid)))
+ (text "S2_SIG: GP15 (yaw)" (at 22 118 0)(effects (font (size 1.2 1.2))(justify left)))
+ (global_label "S2_SIG" (shape input)(at 70 118 0)(effects (font (size 1.0 1.0))(justify left)))
+ (wire (pts (xy 69 118) (xy 70 118)) (stroke (width 0.15)(type solid)))
+ (text "VSERVO" (at 22 122 0)(effects (font (size 1.2 1.2))(justify left)))
+ (global_label "VSERVO" (shape input)(at 70 122 0)(effects (font (size 1.0 1.0))(justify left)))
+ (wire (pts (xy 69 122) (xy 70 122)) (stroke (width 0.15)(type solid)))
+ (text "GND" (at 22 126 0)(effects (font (size 1.2 1.2))(justify left)))
+ (global_label "GND" (shape input)(at 70 126 0)(effects (font (size 1.0 1.0))(justify left)))
+ (wire (pts (xy 69 126) (xy 70 126)) (stroke (width 0.15)(type solid)))
   (sheet_instances (path "/" (page "1"))))

Commit message: Update!
Other:
- company: Skylight Rocketry -> Skylight Industries
- title: WYVERN-E, TVC balance harness (servo rig, Pico) -> GTR70E WYVERN, TVC balance harness (servo rig, Pico)
Changed lines of the file:
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@@
-(kicad_sch (version 20230121) (generator "wyvern4_wiring") (paper "A2")
-  (title_block (title "WYVERN-E, TVC balance harness (servo rig, Pico)") (company "Skylight Rocketry") (rev "4.0"))
+(kicad_sch (version 20230121) (generator "gtr70e_wyvern_wiring") (paper "A2")
+  (title_block (title "GTR70E WYVERN, TVC balance harness (servo rig, Pico)") (company "Skylight Industries") (rev "4.0"))
   (rectangle (start 20 20) (end 84 54) (stroke (width 0.25)(type solid)) (fill (type none)))
  (text "RPi PICO / PICO 2 W, servo-rig DAQ" (at 22 23 0)(effects (font (size 1.6 1.6))(justify left)))
