File: Flight Computer/wiring/WYVERN_E4_tvc_balance_solenoid_harness.kicad_sch (KiCad schematic)
At the start: 0 parts

Commit message: Commit!
Other:
- title: WYVERN-E 4.0 — TVC balance harness (solenoid rig, Pico) -> WYVERN-E — TVC balance harness (solenoid rig, Pico)
Changed lines of the file:
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@@
 (kicad_sch (version 20230121) (generator "wyvern4_wiring") (paper "A2")
-  (title_block (title "WYVERN-E 4.0 — TVC balance harness (solenoid rig, Pico)") (company "Skylight Rocketry") (rev "4.0"))
+  (title_block (title "WYVERN-E — TVC balance harness (solenoid rig, Pico)") (company "Skylight Rocketry") (rev "4.0"))
   (rectangle (start 20 20) (end 84 46) (stroke (width 0.25)(type solid)) (fill (type none)))
   (text "RPi PICO / PICO 2 W — solenoid-rig DAQ" (at 22 23 0)(effects (font (size 1.6 1.6))(justify left)))

Commit message: Update - but the PCB no work :(
Other:
- note added: "RPi PICO / PICO 2 W, solenoid-rig DAQ"
- note removed: "RPi PICO / PICO 2 W — solenoid-rig DAQ"
- title: WYVERN-E — TVC balance harness (solenoid rig, Pico) -> WYVERN-E, TVC balance harness (solenoid rig, Pico)
Changed lines of the file:
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@@
 (kicad_sch (version 20230121) (generator "wyvern4_wiring") (paper "A2")
-  (title_block (title "WYVERN-E — TVC balance harness (solenoid rig, Pico)") (company "Skylight Rocketry") (rev "4.0"))
+  (title_block (title "WYVERN-E, TVC balance harness (solenoid rig, Pico)") (company "Skylight Rocketry") (rev "4.0"))
   (rectangle (start 20 20) (end 84 46) (stroke (width 0.25)(type solid)) (fill (type none)))
-  (text "RPi PICO / PICO 2 W — solenoid-rig DAQ" (at 22 23 0)(effects (font (size 1.6 1.6))(justify left)))
-  (text "3V3: HX711 + BNO085 power" (at 22 28 0)(effects (font (size 1.2 1.2))(justify left)))
-  (global_label "3V3" (shape input)(at 84 28 0)(effects (font (size 1.0 1.0))(justify left)))
-  (wire (pts (xy 83 28) (xy 84 28)) (stroke (width 0.15)(type solid)))
-  (text "GND" (at 22 32 0)(effects (font (size 1.2 1.2))(justify left)))
-  (global_label "GND" (shape input)(at 84 32 0)(effects (font (size 1.0 1.0))(justify left)))
-  (wire (pts (xy 83 32) (xy 84 32)) (stroke (width 0.15)(type solid)))
-  (text "USB: CSV log to host" (at 22 36 0)(effects (font (size 1.2 1.2))(justify left)))
-  (global_label "USB" (shape input)(at 84 36 0)(effects (font (size 1.0 1.0))(justify left)))
-  (wire (pts (xy 83 36) (xy 84 36)) (stroke (width 0.15)(type solid)))
-  (text "GP4/GP5: I2C0 -> BNO085 (gimbal attitude)" (at 22 40 0)(effects (font (size 1.2 1.2))(justify left)))
-  (global_label "GP4/GP5" (shape input)(at 84 40 0)(effects (font (size 1.0 1.0))(justify left)))
-  (wire (pts (xy 83 40) (xy 84 40)) (stroke (width 0.15)(type solid)))
-  (text "GP16-19: solenoid PWM -> 4x IRF520 gate" (at 22 44 0)(effects (font (size 1.2 1.2))(justify left)))
-  (global_label "GP16-19" (shape input)(at 84 44 0)(effects (font (size 1.0 1.0))(justify left)))
-  (wire (pts (xy 83 44) (xy 84 44)) (stroke (width 0.15)(type solid)))
-  (rectangle (start 20 54) (end 76 72) (stroke (width 0.25)(type solid)) (fill (type none)))
-  (text "LOAD CELLS + HX711 x3 (bit-banged)" (at 22 57 0)(effects (font (size 1.6 1.6))(justify left)))
-  (text "Z (axial, 5kg): DT GP10 / SCK GP11" (at 22 62 0)(effects (font (size 1.2 1.2))(justify left)))
-  (global_label "Z (axial, 5kg)" (shape input)(at 76 62 0)(effects (font (size 1.0 1.0))(justify left)))
-  (wire (pts (xy 75 62) (xy 76 62)) (stroke (width 0.15)(type solid)))
-  (text "X (lateral, 1kg): DT GP12 / SCK GP13" (at 22 66 0)(effects (font (size 1.2 1.2))(justify left)))
-  (global_label "X (lateral, 1kg)" (shape input)(at 76 66 0)(effects (font (size 1.0 1.0))(justify left)))
-  (wire (pts (xy 75 66) (xy 76 66)) (stroke (width 0.15)(type solid)))
-  (text "Y (lateral, 1kg): DT GP14 / SCK GP15" (at 22 70 0)(effects (font (size 1.2 1.2))(justify left)))
-  (global_label "Y (lateral, 1kg)" (shape input)(at 76 70 0)(effects (font (size 1.0 1.0))(justify left)))
-  (wire (pts (xy 75 70) (xy 76 70)) (stroke (width 0.15)(type solid)))
-  (rectangle (start 20 80) (end 68 90) (stroke (width 0.25)(type solid)) (fill (type none)))
-  (text "GIMBAL BNO085 (I2C0 0x4A)" (at 22 83 0)(effects (font (size 1.6 1.6))(justify left)))
-  (text "Game Rotation Vector + gyro rate -> deflection from 3-axis load balance" (at 22 88 0)(effects (font (size 1.2 1.2))(justify left)))
-  (global_label "Game Rotation Vector + gyro rate -> deflection from 3-axis load balance" (shape input)(at 68 88 0)(effects (font (size 1.0 1.0))(justify left)))
-  (wire (pts (xy 67 88) (xy 68 88)) (stroke (width 0.15)(type solid)))
-  (rectangle (start 20 98) (end 82 124) (stroke (width 0.25)(type solid)) (fill (type none)))
-  (text "SOLENOIDS x4 via IRF520 (+ 1N4007 flyback EACH)" (at 22 101 0)(effects (font (size 1.6 1.6))(justify left)))
-  (text "PITCH+: GP16" (at 22 106 0)(effects (font (size 1.2 1.2))(justify left)))
-  (global_label "PITCH+" (shape input)(at 82 106 0)(effects (font (size 1.0 1.0))(justify left)))
-  (wire (pts (xy 81 106) (xy 82 106)) (stroke (width 0.15)(type solid)))
-  (text "PITCH-: GP17" (at 22 110 0)(effects (font (size 1.2 1.2))(justify left)))
-  (global_label "PITCH-" (shape input)(at 82 110 0)(effects (font (size 1.0 1.0))(justify left)))
-  (wire (pts (xy 81 110) (xy 82 110)) (stroke (width 0.15)(type solid)))
-  (text "YAW+: GP18" (at 22 114 0)(effects (font (size 1.2 1.2))(justify left)))
-  (global_label "YAW+" (shape input)(at 82 114 0)(effects (font (size 1.0 1.0))(justify left)))
-  (wire (pts (xy 81 114) (xy 82 114)) (stroke (width 0.15)(type solid)))
-  (text "YAW-: GP19" (at 22 118 0)(effects (font (size 1.2 1.2))(justify left)))
-  (global_label "YAW-" (shape input)(at 82 118 0)(effects (font (size 1.0 1.0))(justify left)))
-  (wire (pts (xy 81 118) (xy 82 118)) (stroke (width 0.15)(type solid)))
-  (text "V12: coil supply" (at 22 122 0)(effects (font (size 1.2 1.2))(justify left)))
-  (global_label "V12" (shape input)(at 82 122 0)(effects (font (size 1.0 1.0))(justify left)))
-  (wire (pts (xy 81 122) (xy 82 122)) (stroke (width 0.15)(type solid)))
+ (text "RPi PICO / PICO 2 W, solenoid-rig DAQ" (at 22 23 0)(effects (font (size 1.6 1.6))(justify left)))
+ (text "3V3: HX711 + BNO085 power" (at 22 28 0)(effects (font (size 1.2 1.2))(justify left)))
+ (global_label "3V3" (shape input)(at 84 28 0)(effects (font (size 1.0 1.0))(justify left)))
+ (wire (pts (xy 83 28) (xy 84 28)) (stroke (width 0.15)(type solid)))
+ (text "GND" (at 22 32 0)(effects (font (size 1.2 1.2))(justify left)))
+ (global_label "GND" (shape input)(at 84 32 0)(effects (font (size 1.0 1.0))(justify left)))
+ (wire (pts (xy 83 32) (xy 84 32)) (stroke (width 0.15)(type solid)))
+ (text "USB: CSV log to host" (at 22 36 0)(effects (font (size 1.2 1.2))(justify left)))
+ (global_label "USB" (shape input)(at 84 36 0)(effects (font (size 1.0 1.0))(justify left)))
+ (wire (pts (xy 83 36) (xy 84 36)) (stroke (width 0.15)(type solid)))
+ (text "GP4/GP5: I2C0 -> BNO085 (gimbal attitude)" (at 22 40 0)(effects (font (size 1.2 1.2))(justify left)))
+ (global_label "GP4/GP5" (shape input)(at 84 40 0)(effects (font (size 1.0 1.0))(justify left)))
+ (wire (pts (xy 83 40) (xy 84 40)) (stroke (width 0.15)(type solid)))
+ (text "GP16-19: solenoid PWM -> 4x IRF520 gate" (at 22 44 0)(effects (font (size 1.2 1.2))(justify left)))
+ (global_label "GP16-19" (shape input)(at 84 44 0)(effects (font (size 1.0 1.0))(justify left)))
+ (wire (pts (xy 83 44) (xy 84 44)) (stroke (width 0.15)(type solid)))
+ (rectangle (start 20 54) (end 76 72) (stroke (width 0.25)(type solid)) (fill (type none)))
+ (text "LOAD CELLS + HX711 x3 (bit-banged)" (at 22 57 0)(effects (font (size 1.6 1.6))(justify left)))
+ (text "Z (axial, 5kg): DT GP10 / SCK GP11" (at 22 62 0)(effects (font (size 1.2 1.2))(justify left)))
+ (global_label "Z (axial, 5kg)" (shape input)(at 76 62 0)(effects (font (size 1.0 1.0))(justify left)))
+ (wire (pts (xy 75 62) (xy 76 62)) (stroke (width 0.15)(type solid)))
+ (text "X (lateral, 1kg): DT GP12 / SCK GP13" (at 22 66 0)(effects (font (size 1.2 1.2))(justify left)))
+ (global_label "X (lateral, 1kg)" (shape input)(at 76 66 0)(effects (font (size 1.0 1.0))(justify left)))
+ (wire (pts (xy 75 66) (xy 76 66)) (stroke (width 0.15)(type solid)))
+ (text "Y (lateral, 1kg): DT GP14 / SCK GP15" (at 22 70 0)(effects (font (size 1.2 1.2))(justify left)))
+ (global_label "Y (lateral, 1kg)" (shape input)(at 76 70 0)(effects (font (size 1.0 1.0))(justify left)))
+ (wire (pts (xy 75 70) (xy 76 70)) (stroke (width 0.15)(type solid)))
+ (rectangle (start 20 80) (end 68 90) (stroke (width 0.25)(type solid)) (fill (type none)))
+ (text "GIMBAL BNO085 (I2C0 0x4A)" (at 22 83 0)(effects (font (size 1.6 1.6))(justify left)))
+ (text "Game Rotation Vector + gyro rate -> deflection from 3-axis load balance" (at 22 88 0)(effects (font (size 1.2 1.2))(justify left)))
+ (global_label "Game Rotation Vector + gyro rate -> deflection from 3-axis load balance" (shape input)(at 68 88 0)(effects (font (size 1.0 1.0))(justify left)))
+ (wire (pts (xy 67 88) (xy 68 88)) (stroke (width 0.15)(type solid)))
+ (rectangle (start 20 98) (end 82 124) (stroke (width 0.25)(type solid)) (fill (type none)))
+ (text "SOLENOIDS x4 via IRF520 (+ 1N4007 flyback EACH)" (at 22 101 0)(effects (font (size 1.6 1.6))(justify left)))
+ (text "PITCH+: GP16" (at 22 106 0)(effects (font (size 1.2 1.2))(justify left)))
+ (global_label "PITCH+" (shape input)(at 82 106 0)(effects (font (size 1.0 1.0))(justify left)))
+ (wire (pts (xy 81 106) (xy 82 106)) (stroke (width 0.15)(type solid)))
+ (text "PITCH-: GP17" (at 22 110 0)(effects (font (size 1.2 1.2))(justify left)))
+ (global_label "PITCH-" (shape input)(at 82 110 0)(effects (font (size 1.0 1.0))(justify left)))
+ (wire (pts (xy 81 110) (xy 82 110)) (stroke (width 0.15)(type solid)))
+ (text "YAW+: GP18" (at 22 114 0)(effects (font (size 1.2 1.2))(justify left)))
+ (global_label "YAW+" (shape input)(at 82 114 0)(effects (font (size 1.0 1.0))(justify left)))
+ (wire (pts (xy 81 114) (xy 82 114)) (stroke (width 0.15)(type solid)))
+ (text "YAW-: GP19" (at 22 118 0)(effects (font (size 1.2 1.2))(justify left)))
+ (global_label "YAW-" (shape input)(at 82 118 0)(effects (font (size 1.0 1.0))(justify left)))
+ (wire (pts (xy 81 118) (xy 82 118)) (stroke (width 0.15)(type solid)))
+ (text "V12: coil supply" (at 22 122 0)(effects (font (size 1.2 1.2))(justify left)))
+ (global_label "V12" (shape input)(at 82 122 0)(effects (font (size 1.0 1.0))(justify left)))
+ (wire (pts (xy 81 122) (xy 82 122)) (stroke (width 0.15)(type solid)))
   (sheet_instances (path "/" (page "1"))))

Commit message: Update!
Other:
- company: Skylight Rocketry -> Skylight Industries
- title: WYVERN-E, TVC balance harness (solenoid rig, Pico) -> GTR70E WYVERN, TVC balance harness (solenoid rig, Pico)
Changed lines of the file:
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@@
-(kicad_sch (version 20230121) (generator "wyvern4_wiring") (paper "A2")
-  (title_block (title "WYVERN-E, TVC balance harness (solenoid rig, Pico)") (company "Skylight Rocketry") (rev "4.0"))
+(kicad_sch (version 20230121) (generator "gtr70e_wyvern_wiring") (paper "A2")
+  (title_block (title "GTR70E WYVERN, TVC balance harness (solenoid rig, Pico)") (company "Skylight Industries") (rev "4.0"))
   (rectangle (start 20 20) (end 84 46) (stroke (width 0.25)(type solid)) (fill (type none)))
  (text "RPi PICO / PICO 2 W, solenoid-rig DAQ" (at 22 23 0)(effects (font (size 1.6 1.6))(justify left)))
